File: lm386_stereo_amp.kicad_pcb (KiCad board)
At the start: 2 copper layers, 55 x 65 mm, 33 parts, among them J1 Conn_01x02_Pin, J2 Conn_01x02_Pin, J3 Conn_01x02_Pin, J4 AudioJack3, U1 LM386, U2 LM386

Commit message: place vias
Parts:
- moved G*** 1.02 mm to (128.3, 68.6)
- moved REF** 1.02 mm to (128.3, 74.4)
Routing:
- net GND: vias 0 -> 35
Other:
- board text added: "JLCJLCJLCJLC"
Changed lines of the file:
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@@
       (outputformat 1)
       (mirror false)
-      (drillshape 1)
+      (drillshape 0)
       (scaleselection 1)
-      (outputdirectory "")
+      (outputdirectory "./gerber/")
     )
   )
@@
     (fp_line (start 4.95 3.4) (end 4.95 -2.35)
       (stroke (width 0.1) (type solid)) (layer "F.Fab"))
-    (pad "1" thru_hole roundrect (at 0 0) (size 1.7 2) (drill 1) (layers "*.Cu" "*.Mask") (roundrect_rratio 0.147059)
+    (pad "1" thru_hole roundrect (at 0 0) (size 1.7 2) (drill 1) (layers "*.Cu" "*.Mask") (roundrect_rratio 0.1470588235)
       (net 3 "+9V") (pinfunction "Pin_1") (pintype "passive"))
     (pad "2" thru_hole oval (at 2.5 0) (size 1.7 2) (drill 1) (layers "*.Cu" "*.Mask")
@@
     )
   )
-  (footprint "Library:mcc_logo" locked (layer "F.Cu")
-    (at 127.254 68.58 -90)
+  (footprint "Library:mcc_logo" (layer "F.Cu")
+    (at 128.27 68.58 -90)
     (attr board_only exclude_from_pos_files exclude_from_bom)
     (fp_text reference "G***" (at 0 0 90) (layer "F.SilkS") hide
@@
     )
   )
-  (footprint "Symbol:OSHW-Logo2_7.3x6mm_SilkScreen" locked (layer "F.Cu")
-    (at 127.254 74.422 -90)
+  (footprint "Symbol:OSHW-Logo2_7.3x6mm_SilkScreen" (layer "F.Cu")
+    (at 128.27 74.422 -90)
     (descr "Open Source Hardware Symbol")
     (tags "Logo Symbol OSHW")
@@
     (effects (font (size 1.5 1.5) (thickness 0.3) bold) (justify left bottom))
   )
+  (gr_text "JLCJLCJLCJLC" (at 125.476 55.626 -90) (layer "F.SilkS")
+    (effects (font (size 0.6 0.6) (thickness 0.1) bold) (justify left bottom))
+  )
   (dimension (type aligned) (layer "Eco1.User")
     (pts (xy 179 20) (xy 179 85))
@@
   (segment (start 154.456 31.5) (end 154.456 32.996) (width 0.8) (layer "B.Cu") (net 3))
   (segment (start 156.972 24.638) (end 156.972 27.178) (width 0.8) (layer "B.Cu") (net 3))
+  (via (at 177.5 57) (size 0.8) (drill 0.4) (layers "F.Cu" "B.Cu") (free) (net 4))
+  (via (at 134 73) (size 0.8) (drill 0.4) (layers "F.Cu" "B.Cu") (free) (net 4))
+  (via (at 161 61) (size 0.8) (drill 0.4) (layers "F.Cu" "B.Cu") (free) (net 4))
+  (via (at 149 82) (size 0.8) (drill 0.4) (layers "F.Cu" "B.Cu") (free) (net 4))
+  (via (at 135 54.5) (size 0.8) (drill 0.4) (layers "F.Cu" "B.Cu") (free) (net 4))
+  (via (at 164.5 75) (size 0.8) (drill 0.4) (layers "F.Cu" "B.Cu") (free) (net 4))
+  (via (at 172 83.5) (size 0.8) (drill 0.4) (layers "F.Cu" "B.Cu") (free) (net 4))
+  (via (at 131 83.5) (size 0.8) (drill 0.4) (layers "F.Cu" "B.Cu") (free) (net 4))
+  (via (at 146.5 41) (size 0.8) (drill 0.4) (layers "F.Cu" "B.Cu") (free) (net 4))
+  (via (at 172 21) (size 0.8) (drill 0.4) (layers "F.Cu" "B.Cu") (free) (net 4))
+  (via (at 125 27) (size 0.8) (drill 0.4) (layers "F.Cu" "B.Cu") (free) (net 4))
+  (via (at 131 21) (size 0.8) (drill 0.4) (layers "F.Cu" "B.Cu") (free) (net 4))
+  (via (at 163 32) (size 0.8) (drill 0.4) (layers "F.Cu" "B.Cu") (free) (net 4))
+  (via (at 125.5 51.5) (size 0.8) (drill 0.4) (layers "F.Cu" "B.Cu") (free) (net 4))
+  (via (at 146 54.5) (size 0.8) (drill 0.4) (layers "F.Cu" "B.Cu") (free) (net 4))
+  (via (at 157 35.5) (size 0.8) (drill 0.4) (layers "F.Cu" "B.Cu") (free) (net 4))
+  (via (at 132 25.5) (size 0.8) (drill 0.4) (layers "F.Cu" "B.Cu") (free) (net 4))
+  (via (at 159 21.5) (size 0.8) (drill 0.4) (layers "F.Cu" "B.Cu") (free) (net 4))
+  (via (at 140.5 62.5) (size 0.8) (drill 0.4) (layers "F.Cu" "B.Cu") (free) (net 4))
+  (via (at 177.5 78) (size 0.8) (drill 0.4) (layers "F.Cu" "B.Cu") (free) (net 4))
+  (via (at 175.5 38.5) (size 0.8) (drill 0.4) (layers "F.Cu" "B.Cu") (free) (net 4))
+  (via (at 164 46.5) (size 0.8) (drill 0.4) (layers "F.Cu" "B.Cu") (free) (net 4))
+  (via (at 155 64.5) (size 0.8) (drill 0.4) (layers "F.Cu" "B.Cu") (free) (net 4))
+  (via (at 174.5 65) (size 0.8) (drill 0.4) (layers "F.Cu" "B.Cu") (free) (net 4))
+  (via (at 145.5 34.5) (size 0.8) (drill 0.4) (layers "F.Cu" "B.Cu") (free) (net 4))
+  (via (at 151 41) (size 0.8) (drill 0.4) (layers "F.Cu" "B.Cu") (free) (net 4))
+  (via (at 125 78) (size 0.8) (drill 0.4) (layers "F.Cu" "B.Cu") (free) (net 4))
+  (via (at 132.5 35) (size 0.8) (drill 0.4) (layers "F.Cu" "B.Cu") (free) (net 4))
+  (via (at 174 31.5) (size 0.8) (drill 0.4) (layers "F.Cu" "B.Cu") (free) (net 4))
+  (via (at 135.5 47) (size 0.8) (drill 0.4) (layers "F.Cu" "B.Cu") (free) (net 4))
+  (via (at 161 27.5) (size 0.8) (drill 0.4) (layers "F.Cu" "B.Cu") (free) (net 4))
+  (via (at 177.5 27) (size 0.8) (drill 0.4) (layers "F.Cu" "B.Cu") (free) (net 4))
+  (via (at 146 48) (size 0.8) (drill 0.4) (layers "F.Cu" "B.Cu") (free) (net 4))
+  (via (at 148.5 78) (size 0.8) (drill 0.4) (layers "F.Cu" "B.Cu") (free) (net 4))
+  (via (at 135.5 66) (size 0.8) (drill 0.4) (layers "F.Cu" "B.Cu") (free) (net 4))
   (segment (start 147.558 31.5) (end 147.558 37.322) (width 0.8) (layer "F.Cu") (net 5))
   (segment (start 147.558 37.322) (end 147.574 37.338) (width 0.8) (layer "F.Cu") (net 5))

Commit message: fix input wire
Parts:
- J1: footprint TerminalBlock:TerminalBlock_bornier-2_P5.08mm -> Connector_JST:JST_XH_B2B-XH-A_1x02_P2.50mm_Vertical
- J2: value Conn_01x02_Pin -> AudioJack3; footprint Connector_JST:JST_XH_B2B-XH-A_1x02_P2.50mm_Vertical -> Connector_Audio:Jack_3.5mm_Switronic_ST-005-G_horizontal
- J4: value AudioJack3 -> Conn_01x02_Pin; footprint Connector_Audio:Jack_3.5mm_Switronic_ST-005-G_horizontal -> TerminalBlock:TerminalBlock_bornier-2_P5.08mm
- moved J4 58.6 mm to (169.9, 75.1), turned to 90 degrees
- moved J1 50.6 mm to (165.6, 24.6), turned to 0 degrees
- moved J2 26.0 mm to (139.6, 24.9), turned to -90 degrees
Connections:
- C12 pad 2: Net-(J1-Pin_2) -> Net-(J4-Pin_2)
- J1 pad 1: GND -> +9V
- J1 pad 2: Net-(J1-Pin_2) -> GND
- RV1 pad 1: Net-(J4-PadR) -> GND
- RV1 pad 3: GND -> Net-(J2-PadR)
- RV1 pad 4: Net-(J4-PadT) -> GND
- RV1 pad 6: GND -> Net-(J2-PadT)
Routing:
- net Net-(J4-PadT): track 47.0 -> 0.00 mm
- net Net-(J2-PadT): track 0.00 -> 46.1 mm
- net Net-(J2-PadR): track 0.00 -> 41.0 mm
- net Net-(J4-PadR): track 31.9 -> 0.00 mm
- net Net-(J4-Pin_2): track 0.00 -> 8.03 mm
- net Net-(J1-Pin_2): track 8.03 -> 0.00 mm
- net Net-(C8-Pad2): track 33.3 -> 30.1 mm
- net Net-(C1-Pad2): track 14.8 -> 13.4 mm
- net GND: vias 35 -> 33
Other:
- board text added: "-Left+"
- board text added: "-Right+"
- board text removed: "Left"
- board text removed: "Right"

Commit message: up to date
Changed lines of the file:
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@@
     (fp_line (start 4.95 3.4) (end 4.95 -2.35)
       (stroke (width 0.1) (type solid)) (layer "F.Fab"))
-    (pad "1" thru_hole roundrect (at 0 0) (size 1.7 2) (drill 1) (layers "*.Cu" "*.Mask") (roundrect_rratio 0.147059)
+    (pad "1" thru_hole roundrect (at 0 0) (size 1.7 2) (drill 1) (layers "*.Cu" "*.Mask") (roundrect_rratio 0.1470588235)
       (net 3 "+9V") (pinfunction "Pin_1") (pintype "passive"))
     (pad "2" thru_hole oval (at 2.5 0) (size 1.7 2) (drill 1) (layers "*.Cu" "*.Mask")
@@
     (property "ki_keywords" "audio jack receptacle stereo headphones phones TRS connector")
     (attr through_hole)
-    (fp_text reference "J2" (at 0 -4.5 90) (layer "F.SilkS")
+    (fp_text reference "J2" (at 1.166 -4.917 -180) (layer "F.SilkS")
         (effects (font (size 1 1) (thickness 0.15)))
     )
@@
         (effects (font (size 1 1) (thickness 0.15)))
     )
-    (fp_text user "${REFERENCE}" (at 1.27 2.794) (layer "F.Fab")
+    (fp_text user "${REFERENCE}" (at 1.172 3.81) (layer "F.Fab")
         (effects (font (size 1 1) (thickness 0.15)))
     )
