File: lm386_stereo_amp.kicad_sch (KiCad schematic)
At the start: 31 parts, among them J1 Conn_01x02_Pin, J2 AudioJack3, J2 Conn_01x02_Pin, U1 LM386

Commit message: fix input wire
Connections:
- net GND: now also RV1.1, RV1.4; no longer RV1.3, RV1.6
- net at J2.R: now also RV1.3; no longer RV1.1
- net at J2.T: now also RV1.6; no longer RV1.4
Changed lines of the file:
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@@
+    (stroke (width 0) (type default))
+  )
+  (wire (pts (xy 53.34 114.935) (xy 49.53 111.125))
     (stroke (width 0) (type default))
   )
@@
     (stroke (width 0) (type default))
   )
+  (wire (pts (xy 86.36 118.745) (xy 77.47 118.745))
+    (stroke (width 0) (type default))
+  )
   (wire (pts (xy 106.045 97.155) (xy 113.03 97.155))
     (stroke (width 0) (type default))
@@
     (stroke (width 0) (type default))
   )
-  (wire (pts (xy 86.36 128.27) (xy 86.36 114.935))
+  (wire (pts (xy 86.36 128.27) (xy 86.36 118.745))
     (stroke (width 0) (type default))
   )
@@
     (stroke (width 0) (type default))
   )
-  (wire (pts (xy 58.42 102.235) (xy 49.53 111.125))
+  (wire (pts (xy 40.64 108.585) (xy 52.07 108.585))
     (stroke (width 0) (type default))
   )
@@
     (stroke (width 0) (type default))
   )
-  (wire (pts (xy 86.36 109.855) (xy 77.47 118.745))
-    (stroke (width 0) (type default))
-  )
   (wire (pts (xy 132.08 107.315) (xy 132.08 109.855))
     (stroke (width 0) (type default))
   )
+  (wire (pts (xy 52.07 108.585) (xy 58.42 102.235))
+    (stroke (width 0) (type default))
+  )
   (wire (pts (xy 158.75 130.81) (xy 166.37 130.81))
     (stroke (width 0) (type default))
@@
     (stroke (width 0) (type default))
   )
-  (wire (pts (xy 86.36 97.155) (xy 86.36 109.855))
+  (wire (pts (xy 86.36 97.155) (xy 86.36 106.045))
     (stroke (width 0) (type default))
   )
@@
     (stroke (width 0) (type default))
   )
-  (wire (pts (xy 86.36 114.935) (xy 77.47 106.045))
-    (stroke (width 0) (type default))
-  )
   (wire (pts (xy 126.365 80.645) (xy 126.365 75.565))
     (stroke (width 0) (type default))
   )
-  (wire (pts (xy 40.64 108.585) (xy 49.53 108.585))
-    (stroke (width 0) (type default))
-  )
   (wire (pts (xy 116.205 80.645) (xy 121.285 80.645))
     (stroke (width 0) (type default))
   )
-  (wire (pts (xy 55.88 114.935) (xy 72.39 114.935))
+  (wire (pts (xy 53.34 114.935) (xy 72.39 114.935))
+    (stroke (width 0) (type default))
+  )
+  (wire (pts (xy 77.47 106.045) (xy 86.36 106.045))
     (stroke (width 0) (type default))
   )
@@
   )
   (wire (pts (xy 131.445 68.58) (xy 131.445 73.025))
-    (stroke (width 0) (type default))
-  )
-  (wire (pts (xy 49.53 108.585) (xy 55.88 114.935))
     (stroke (width 0) (type default))
   )
@@
     )
   )
-  (symbol (lib_id "Device:R_Potentiometer_Dual") (at 74.93 112.395 270) (unit 1)
+  (symbol (lib_id "Device:R_Potentiometer_Dual") (at 74.93 112.395 270) (mirror x) (unit 1)
     (in_bom yes) (on_board yes) (dnp no)
-    (property "Reference" "RV1" (at 70.485 111.125 90)
+    (property "Reference" "RV1" (at 70.485 113.665 90)
       (effects (font (size 1.27 1.27)) (justify right))
     )
-    (property "Value" "R_Potentiometer_Dual" (at 70.485 113.665 90)
+    (property "Value" "R_Potentiometer_Dual" (at 70.485 111.125 90)
       (effects (font (size 1.27 1.27)) (justify right))
     )
-    (property "Footprint" "Potentiometer_THT:Potentiometer_Alps_RK097_Dual_Horizontal" (at 73.025 118.745 0)
-      (effects (font (size 1.27 1.27)) hide)
-    )
-    (property "Datasheet" "~" (at 73.025 118.745 0)
-      (effects (font (size 1.27 1.27)) hide)
-    )
+    (property "Footprint" "Potentiometer_THT:Potentiometer_Alps_RK097_Dual_Horizontal" (at 73.025 106.045 0)
+      (effects (font (size 1.27 1.27)) hide)
+    )
+    (property "Datasheet" "~" (at 73.025 106.045 0)
+      (effects (font (size 1.27 1.27)) hide)
+    )

Commit message: up to date
Parts:
- RV1: value R_Potentiometer_Dual -> 10kΩ
Changed lines of the file:
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@@
       (effects (font (size 1.27 1.27)) (justify right))
     )
-    (property "Value" "R_Potentiometer_Dual" (at 70.485 111.125 90)
+    (property "Value" "10kΩ" (at 70.485 111.125 90)
       (effects (font (size 1.27 1.27)) (justify right))
     )
